Commit message: Update package references from 'description' to 'sigyn_description' in URDF files
Co-authored-by: wimblerobotics <44647075+wimblerobotics@users.noreply.github.com>

File: urdf/gripper_assembly.urdf.xacro (robot description, xacro)
@@ -1,5 +1,5 @@
 <?xml version="1.0"?>
 <robot xmlns:xacro="http://ros.org/wiki/xacro" name="Sigyn">
-    <xacro:include filename="$(find description)/urdf/gripper_assembly_properties.urdf.xacro" />
+    <xacro:include filename="$(find sigyn_description)/urdf/gripper_assembly_properties.urdf.xacro" />
     <xacro:colorize_link color="0.95 1.0 0.95 1.0" name="evelator_pole">
         <foo>

File: urdf/oakd.urdf.xacro (robot description, xacro)
@@ -27,5 +27,5 @@
         <origin rpy="0 0 0" xyz="0 0 0" />
         <geometry>
-          <mesh filename="package://description/meshes/OAK-D.dae" />
+          <mesh filename="package://sigyn_description/meshes/OAK-D.dae" />
         </geometry>
         <material name="mat">

File: urdf/ros2_control.xacro (robot description, xacro)
@@ -123,6 +123,6 @@
   <gazebo>
     <plugin name="gz_ros2_control::GazeboSimROS2ControlPlugin" filename="libgz_ros2_control-system.so">
-      <parameters>$(find description)/config/my_controllers.yaml</parameters>
-      <parameters>$(find description)/config/gaz_ros2_ctl_use_sim.yaml</parameters>
+      <parameters>$(find sigyn_description)/config/my_controllers.yaml</parameters>
+      <parameters>$(find sigyn_description)/config/gaz_ros2_ctl_use_sim.yaml</parameters>
     </plugin>
   </gazebo>

File: urdf/sigyn.urdf.xacro (robot description, xacro)
@@ -4,15 +4,15 @@
   <xacro:arg name="sim_mode" default="false" />
   <xacro:arg name="do_top_lidar" default="true" />
-  <xacro:include filename="$(find description)/urdf/common_macros.xacro" />
-  <xacro:include filename="$(find description)/urdf/inertials.xacro" />
+  <xacro:include filename="$(find sigyn_description)/urdf/common_macros.xacro" />
+  <xacro:include filename="$(find sigyn_description)/urdf/inertials.xacro" />
   <xacro:property name="props" value="${xacro.load_yaml('sigyn_config.yaml')}" />
-  <xacro:include filename="$(find description)/urdf/sigyn_base_macro.urdf.xacro" />
-  <xacro:include filename="$(find description)/urdf/sigyn_caster_wheel_macro.urdf.xacro" />
-  <xacro:include filename="$(find description)/urdf/sigyn_wheels_macro.urdf.xacro" />
+  <xacro:include filename="$(find sigyn_description)/urdf/sigyn_base_macro.urdf.xacro" />
+  <xacro:include filename="$(find sigyn_description)/urdf/sigyn_caster_wheel_macro.urdf.xacro" />
+  <xacro:include filename="$(find sigyn_description)/urdf/sigyn_wheels_macro.urdf.xacro" />
   <xacro:unless value="$(arg sim_mode)">
-    <xacro:include filename="$(find description)/urdf/depthai_macro.urdf.xacro" />
+    <xacro:include filename="$(find sigyn_description)/urdf/depthai_macro.urdf.xacro" />
   </xacro:unless>
   <xacro:unless value="$(arg sim_mode)">
-    <xacro:include filename="$(find description)/urdf/oakd.urdf.xacro" />
+    <xacro:include filename="$(find sigyn_description)/urdf/oakd.urdf.xacro" />
   </xacro:unless>
   <xacro:if value="$(arg use_ros2_control)">
@@ -28,5 +28,5 @@
   <!-- Make the caster wheel -->
   <xacro:caster_wheel config="${props}" />
-  <xacro:include filename="$(find description)/urdf/ld06.urdf.xacro" />
+  <xacro:include filename="$(find sigyn_description)/urdf/ld06.urdf.xacro" />
   <!-- LiDAR configuration: if do_top_lidar=true, use both top_lidar and cup_lidar as-is.
        if do_top_lidar=false, create only a top_lidar at the cup_lidar origin so downstream
@@ -45,6 +45,6 @@
     </xacro:ld06>
   </xacro:unless>
-  <xacro:include filename="$(find description)/urdf/gazebo.urdf.xacro" />
-  <xacro:include filename="$(find description)/urdf/gripper_assembly.urdf.xacro" />
+  <xacro:include filename="$(find sigyn_description)/urdf/gazebo.urdf.xacro" />
+  <xacro:include filename="$(find sigyn_description)/urdf/gripper_assembly.urdf.xacro" />
   <joint name="base_link_to_elevator_pole" type="fixed">
     <origin xyz="-0.16 -0.015 ${0.3 + (elevator_pole_height/2)}" rpy="0 0 0" />
@@ -138,8 +138,8 @@
   </joint>
   <link name="imu_1" />
-  <xacro:include filename="$(find description)/urdf/vl53l0x.xacro" />
+  <xacro:include filename="$(find sigyn_description)/urdf/vl53l0x.xacro" />
   <!-- Simulation cameras for Can Do Challenge -->
   <xacro:if value="$(arg sim_mode)">
-    <xacro:include filename="$(find description)/urdf/sim_cameras.urdf.xacro" />
+    <xacro:include filename="$(find sigyn_description)/urdf/sim_cameras.urdf.xacro" />
     <xacro:oakd_sim_camera parent_link="base_link"/>
     <xacro:pi_camera_sim parent_link="parallel_gripper_base_plate"/>

Commit message: Fix typo: evelator_pole -> elevator_pole
Co-authored-by: wimblerobotics <44647075+wimblerobotics@users.noreply.github.com>

File: urdf/gripper_assembly.urdf.xacro (robot description, xacro)
@@ -2,5 +2,5 @@
 <robot xmlns:xacro="http://ros.org/wiki/xacro" name="Sigyn">
     <xacro:include filename="$(find sigyn_description)/urdf/gripper_assembly_properties.urdf.xacro" />
-    <xacro:colorize_link color="0.95 1.0 0.95 1.0" name="evelator_pole">
+    <xacro:colorize_link color="0.95 1.0 0.95 1.0" name="elevator_pole">
         <foo>
             <visual>
@@ -8,5 +8,5 @@
                     <box size="${elevator_pole_length} ${elevator_pole_width} ${elevator_pole_height}" />
                 </geometry>
-                <material name="evelator_pole"/>
+                <material name="elevator_pole"/>
             </visual>
             <collision>
@@ -36,5 +36,5 @@
     <joint name="elevator_pole_to_conveyor_belt" type="fixed">
         <origin xyz="0.0 ${((elevator_pole_width/2)+0.0005)} 0.0" rpy="0 0 0" />
-        <parent link="evelator_pole" />
+        <parent link="elevator_pole" />
         <child link="conveyor_belt" />
         <axis xyz="0 0 1" />
@@ -58,5 +58,5 @@
     <joint name="elevator_pole_to_elevator_connector_plate" type="prismatic">
         <origin xyz="0.0 ${(elevator_pole_width/2)+(elevator_connector_plate_height/2)} ${(-elevator_pole_height/2)+(elevator_connector_plate_width/2)}" rpy="0 0 0" />
-        <parent link="evelator_pole" />
+        <parent link="elevator_pole" />
         <child link="elevator_connector_plate" />
         <limit lower="0.15" upper="${elevator_pole_height-(elevator_connector_plate_width)}" effort="50" velocity="0.5" />

File: urdf/sigyn.urdf.xacro (robot description, xacro)
@@ -50,5 +50,5 @@
     <origin xyz="-0.16 -0.015 ${0.3 + (elevator_pole_height/2)}" rpy="0 0 0" />
     <parent link="base_link" />
-    <child link="evelator_pole" />
+    <child link="elevator_pole" />
   </joint>
   <!-- <xacro:oakd_link mount_point="elevator_top" /> -->
