Commit message: Add Mac Silicon compatibility with on_a_mac parameter
- Add on_a_mac boolean parameter to handle platform-specific differences
- Conditionally use ray sensor (Mac) vs gpu_lidar (native) for LD06 lidar
- Update launch file to pass on_a_mac parameter to xacro processing
- Fix package name references: description -> sigyn_description
- Document on_a_mac parameter usage in README
- Add launch examples for Mac Silicon

This resolves GPU passthrough issues in Parallels VMs by using
software-compatible ray sensor when on_a_mac=true.

File: urdf/ld06.urdf.xacro (robot description, xacro)
@@ -1,5 +1,5 @@
 <?xml version="1.0"?>
 <robot xmlns:xacro="http://ros.org/wiki/xacro" name="ld06">
-  <xacro:macro name="ld06" params="lidar_prefix topic_name:=scan *joint_pose">
+  <xacro:macro name="ld06" params="lidar_prefix topic_name:=scan on_a_mac:=false *joint_pose">
     <material name="ld06_${lidar_prefix}_grey">
       <color rgba="0.3 0.3 0.3 1" />
@@ -67,32 +67,9 @@
     <gazebo reference="lidar_frame_${lidar_prefix}">
       <material>Gazebo/Black</material>
-      <sensor name="lidar_frame_${lidar_prefix}" type="gpu_lidar">
-        <visualize>true</visualize>
-        <update_rate>10</update_rate>
-        <lidar>
-          <scan>
-            <horizontal>
-              <samples>450</samples>
-              <resolution>1</resolution>
-              <min_angle>-3.14159</min_angle>
-              <max_angle>3.14159</max_angle>
-            </horizontal>
-            <vertical>
-              <samples>1</samples>
-              <resolution>1</resolution>
-              <min_angle>0</min_angle>
-              <max_angle>0</max_angle>
-            </vertical>
-          </scan>
-          <range>
-            <min>0.3</min>
-            <max>12.0</max>
-          </range>
-          <noise>
-            <type>gaussian</type>
-            <mean>0.0</mean>
-            <stddev>0.01</stddev>
-          </noise>
-          <!-- Add ray filtering to handle self-collisions -->
+      <!-- Use ray sensor type on Mac Silicon (software GL), gpu_lidar elsewhere -->
+      <xacro:if value="${on_a_mac}">
+        <sensor name="lidar_frame_${lidar_prefix}" type="ray">
+          <visualize>true</visualize>
+          <update_rate>10</update_rate>
           <ray>
             <scan>
@@ -108,18 +85,80 @@
               <max>12.0</max>
             </range>
+            <noise>
+              <type>gaussian</type>
+              <mean>0.0</mean>
+              <stddev>0.01</stddev>
+            </noise>
           </ray>
-        </lidar>
-        <topic>${topic_name}</topic>
-        <gz_frame_id>lidar_beam_${lidar_prefix}</gz_frame_id>
-      </sensor>
-      <!-- Use correct Gazebo Garden/Harmonic plugin -->
-      <plugin name="gazebo_ros_laser_controller" filename="libgazebo_ros_gpu_laser.so">
-        <ros>
-          <namespace></namespace>
-          <remapping>~/out:=${topic_name}</remapping>
-        </ros>
-        <output_type>sensor_msgs/LaserScan</output_type>
-        <frame_name>lidar_beam_${lidar_prefix}</frame_name>
-      </plugin>
+          <topic>${topic_name}</topic>
+          <gz_frame_id>lidar_beam_${lidar_prefix}</gz_frame_id>
+        </sensor>
+        <!-- Use ray-based plugin for Mac Silicon compatibility -->
+        <plugin name="gazebo_ros_laser_controller" filename="libgazebo_ros_ray_sensor.so">
+          <ros>
+            <namespace></namespace>
+            <remapping>~/out:=${topic_name}</remapping>
+          </ros>
+          <output_type>sensor_msgs/LaserScan</output_type>
+          <frame_name>lidar_beam_${lidar_prefix}</frame_name>
+        </plugin>
+      </xacro:if>
+      <xacro:unless value="${on_a_mac}">
+        <sensor name="lidar_frame_${lidar_prefix}" type="gpu_lidar">
+          <visualize>true</visualize>
+          <update_rate>10</update_rate>
+          <lidar>
+            <scan>
+              <horizontal>
+                <samples>450</samples>
+                <resolution>1</resolution>
+                <min_angle>-3.14159</min_angle>
+                <max_angle>3.14159</max_angle>
+              </horizontal>
+              <vertical>
+                <samples>1</samples>
+                <resolution>1</resolution>
+                <min_angle>0</min_angle>
+                <max_angle>0</max_angle>
+              </vertical>
+            </scan>
+            <range>
+              <min>0.3</min>
+              <max>12.0</max>
+            </range>
+            <noise>
+              <type>gaussian</type>
+              <mean>0.0</mean>
+              <stddev>0.01</stddev>
+            </noise>
+            <!-- Add ray filtering to handle self-collisions -->
+            <ray>
+              <scan>
+                <horizontal>
+                  <samples>450</samples>
+                  <resolution>1</resolution>
+                  <min_angle>-3.14159</min_angle>
+                  <max_angle>3.14159</max_angle>
+                </horizontal>
+              </scan>
+              <range>
+                <min>0.3</min>
+                <max>12.0</max>
+              </range>
+            </ray>
+          </lidar>
+          <topic>${topic_name}</topic>
+          <gz_frame_id>lidar_beam_${lidar_prefix}</gz_frame_id>
+        </sensor>
+        <!-- Use GPU-accelerated plugin for better performance -->
+        <plugin name="gazebo_ros_laser_controller" filename="libgazebo_ros_gpu_laser.so">
+          <ros>
+            <namespace></namespace>
+            <remapping>~/out:=${topic_name}</remapping>
+          </ros>
+          <output_type>sensor_msgs/LaserScan</output_type>
+          <frame_name>lidar_beam_${lidar_prefix}</frame_name>
+        </plugin>
+      </xacro:unless>
     </gazebo>
   </xacro:macro>

File: urdf/sigyn.urdf.xacro (robot description, xacro)
@@ -4,4 +4,5 @@
   <xacro:arg name="sim_mode" default="false" />
   <xacro:arg name="do_top_lidar" default="true" />
+  <xacro:arg name="on_a_mac" default="false" />
   <xacro:include filename="$(find sigyn_description)/urdf/common_macros.xacro" />
   <xacro:include filename="$(find sigyn_description)/urdf/inertials.xacro" />
@@ -33,13 +34,13 @@
        code continues to use the 'top_lidar' name and 'scan' topic. -->
   <xacro:if value="$(arg do_top_lidar)">
-    <xacro:ld06 lidar_prefix="top_lidar" topic_name="scan">
+    <xacro:ld06 lidar_prefix="top_lidar" topic_name="scan" on_a_mac="$(arg on_a_mac)">
       <origin xyz="${0.155-0.34} 0 ${1.485}" rpy="0 0 0" />
     </xacro:ld06>
-    <xacro:ld06 lidar_prefix="cup_lidar" topic_name="scan_cup">
+    <xacro:ld06 lidar_prefix="cup_lidar" topic_name="scan_cup" on_a_mac="$(arg on_a_mac)">
       <origin xyz="0.155 0 0.300" rpy="0 0 -${pi / 2}" />
     </xacro:ld06>
   </xacro:if>
   <xacro:unless value="$(arg do_top_lidar)">
-    <xacro:ld06 lidar_prefix="top_lidar" topic_name="scan">
+    <xacro:ld06 lidar_prefix="top_lidar" topic_name="scan" on_a_mac="$(arg on_a_mac)">
       <origin xyz="0.155 0 0.300" rpy="0 0 -${pi / 2}" />
     </xacro:ld06>
