Commit message: Fix OAK-D visual mesh orientation

File: urdf/oakd.urdf.xacro (robot description, xacro)
@@ -37,5 +37,5 @@
       <parent link="oak" />
       <child link="oak_model_origin" />
-      <origin rpy="1.5708 0 1.5708" xyz="0 0 0" />
+      <origin rpy="0 0 0" xyz="0 0 0" />
     </joint> <!-- IMU -->
     <link name="oak_imu_frame" />
